File: SMDModelF/SMDModelF.kicad_pcb (KiCad board)
At the start: 2 copper layers, 143.3 x 41.8 mm, 44 parts, among them J1 Model F Ribbon Cable, J2 PadsToShort, J3 EXPANSION HEADER, J5 Conn_01x03, J7 Conn_01x05, U1 MCP4921-E, U2 LM339A, U3 74AHC595, U4 74AHC595, U5 ProMicro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

Commit message: PCB file: updated footprints and references to 3d parts.
Parts:
- J7: footprint Connector_PinHeader_2.54mm:PinHeader_1x05_P2.54mm_Vertical -> TH-XWhatsIt:PinHeader_1x05_P2.54mm_Vertical_no3d
